File: hardware/preamp/preamp.sch (KiCad schematic (older format))
At the start: 27 parts, among them P1 1702473, P2 BARREL_JACK, P3 SMA, U1 OPA2365, U2 NCP1117ST50T3G, Y1 60kHz

Commit message: Moved footprint library into hardware folder
Parts:
- C6: footprint wwvb-receiver:TZY2 -> radio-clock:TZY2
- P1: footprint wwvb-receiver:1702473 -> radio-clock:1702473
- P2: footprint wwvb-receiver:PJ-002AH-SMT-TR -> radio-clock:PJ-002AH-SMT-TR
- P3: footprint wwvb-receiver:142-0701-801 -> radio-clock:142-0701-801
Changed lines of the file:
@@
 F 0 "P3" H 8160 3670 50  0000 C CNN
 F 1 "SMA" H 8250 3400 50  0000 C CNN
-F 2 "wwvb-receiver:142-0701-801" H 8150 3550 50  0001 C CNN
+F 2 "radio-clock:142-0701-801" H 8150 3550 50  0001 C CNN
 F 3 "" H 8150 3550 50  0000 C CNN
 F 4 "DigiKey" H 8150 3550 60  0001 C CNN "Source"
@@
 F 0 "P1" H 2350 3650 50  0000 C CNN
 F 1 "1702473" H 2350 3350 50  0000 C CNN
-F 2 "wwvb-receiver:1702473" H 2350 3500 50  0001 C CNN
+F 2 "radio-clock:1702473" H 2350 3500 50  0001 C CNN
 F 3 "" H 2350 3500 50  0000 C CNN
 F 4 "DigiKey" H 2350 3500 60  0001 C CNN "Source"
@@
 F 0 "P2" H 2650 6250 50  0000 C CNN
 F 1 "BARREL_JACK" H 2650 5800 50  0000 C CNN
-F 2 "wwvb-receiver:PJ-002AH-SMT-TR" H 2650 6000 50  0001 C CNN
+F 2 "radio-clock:PJ-002AH-SMT-TR" H 2650 6000 50  0001 C CNN
 F 3 "" H 2650 6000 50  0000 C CNN
 F 4 "DigiKey" H 2650 6000 60  0001 C CNN "Source"
@@
 F 0 "C6" V 5000 3300 50  0000 L CNN
 F 1 "0.5p-1p" V 5300 3200 50  0000 L CNN
-F 2 "wwvb-receiver:TZY2" H 5150 3350 50  0001 C CNN
+F 2 "radio-clock:TZY2" H 5150 3350 50  0001 C CNN
 F 3 "" H 5150 3350 50  0000 C CNN
 F 4 "DigiKey" H 5150 3350 60  0001 C CNN "Source"
