File: hardware/clock/clock.sch (KiCad schematic (older format))
At the start: 22 parts

Commit message: Working on schematic
Parts:
- added U?: HV5522PG, symbol HV5522PG
Changed lines of the file:
@@
 	7050 9000 7050 9050
 Connection ~ 7050 9000
+$Comp
+L HV5522PG U?
+U 1 1 58E01DBF
+P 5650 3950
+F 0 "U?" H 5250 5650 60  0000 C CNN
+F 1 "HV5522PG" H 5900 2250 60  0000 C CNN
+F 2 "" H 5650 3950 60  0001 C CNN
+F 3 "" H 5650 3950 60  0001 C CNN
+	1    5650 3950
+	1    0    0    -1
+$EndComp
 $EndSCHEMATC
