File: hardware/main-board/main-board.sch (KiCad schematic (older format))
At the start: 23 parts

Commit message: Working on tube board schematic
Connections:
- net labels added: HT
- net labels removed: VDD
Changed lines of the file:
@@
 LIBS:Zilog
 LIBS:radio-clock
-LIBS:clock-cache
+LIBS:main-board-cache
 EELAYER 25 0
 EELAYER END
@@
 Wire Wire Line
 	3950 8000 3950 7950
-$Comp
-L VDD #PWR?
-U 1 1 58DFBBAC
-P 8050 8050
-F 0 "#PWR?" H 8050 7900 50  0001 C CNN
-F 1 "VDD" H 8050 8200 50  0000 C CNN
-F 2 "" H 8050 8050 50  0001 C CNN
-F 3 "" H 8050 8050 50  0001 C CNN
-	1    8050 8050
-	1    0    0    -1
-$EndComp
 Connection ~ 8050 8150
 Wire Wire Line
@@
 	1    0    0    -1
 $EndComp
+$Comp
+L HT #PWR?
+U 1 1 58E110D4
+P 8050 8050
+F 0 "#PWR?" H 8050 8170 50  0001 C CNN
+F 1 "HT" H 8050 8140 50  0000 C CNN
+F 2 "" H 8050 8050 50  0001 C CNN
+F 3 "" H 8050 8050 50  0001 C CNN
+	1    8050 8050
+	1    0    0    -1
+$EndComp

Commit message: Working on main board schematic
Parts:
- removed U?: HV5522PG, symbol HV5522PG
- added BT?: 3.7V LION, symbol Battery_Cell
- added C?: 0.1u, symbol C
- added C?: 10u, symbol C
- added C? (x2): 1u, symbol C
- added C?: 0.01u, symbol C
- added C?: 0.1u, Capacitors_SMD:C_0603, symbol C
- added C? (x2): C, symbol C
- added D?: LED, symbol LED
- added D? (x2): D, symbol D
- added J? (x2): CONN_01X10, radio-clock:8-188275-0, symbol CONN_01X10
- added J?: CONN_02X05, symbol CONN_02X05
- added J?: SMA, symbol CONN_COAXIAL
- added L?: FERRITE, symbol L_Core_Ferrite
- added Q? (x5): DDTD113ZC, TO_SOT_Packages_SMD:SOT-23, symbol Q_NPN_BEC
- added R?: R, symbol R
- added R? (x4): 10k, Resistors_SMD:R_0805, symbol R
- added U?: LD1117S33TR, TO_SOT_Packages_SMD:SOT-223, symbol LD1117S33TR
- added U?: FGPMMOPA6H, symbol FGPMMOPA6H
- added Y?: 8MHz, symbol Crystal
- C?: value 100n -> 0.1u
- R?: value R -> 10k
Connections:
- net labels added: +5V, DISP_BL, DISP_CLK, DISP_DATA, DISP_LE, GPS_PPS, GPS_RESET, GPS_RX, GPS_TX, HV_EN, NRST, SWCLK, SWDIO, SWO
- wire segments 78 -> 165
- no-connect marks 0 -> 4
Other:
- moved on the sheet: C?, D?, F?, J?, L?, Q?, R?, U?

Commit message: Working on main board schematic
Parts:
- removed D? (x2): D, symbol D
- added D? (x6): LED_RABG, symbol LED_RABG
- added D?: LED, symbol LED
- added JP?: Jumper_NO_Small, symbol Jumper_NO_Small
- added Q? (x3): DDTD113ZC, TO_SOT_Packages_SMD:SOT-23, symbol Q_NPN_BEC
- added R? (x2): 10k, symbol R
- added R? (x19): R, symbol R
Connections:
- net labels added: BOOT0, DGB_LED, JTDI, LED_BLU, LED_GRN, LED_RED, NJTRST, SWCLK/JTCK, SWDIO/JTMS, SWO/JTDO, USB_VBUS
- net labels removed: +5V, SWCLK, SWDIO, SWO
- wire segments 165 -> 235
- no-connect marks 4 -> 3
Other:
- moved on the sheet: C?, D?, F?, J?, L?, Q?, R?, U?

Commit message: Working on main board schematic
Parts:
- removed C?: 0.1u, symbol C
- removed C?: 0.1u, Capacitors_SMD:C_0603, symbol C
- removed R? (x17): R, symbol R
- removed R?: 10k, symbol R
- removed U?: STM32F302K8, symbol STM32F302K8
- added C1, C7: 0.1u, Capacitors_SMD:C_0805, symbol C
- added C11, C12: 0.1u, Capacitors_SMD:C_0603, symbol C
- added J10, J11, J12, J7, J8, J9: TP, Measurement_Points:Measurement_Point_Round-SMD-Pad_Big, symbol TEST_1P
- added R11, R12, R14, R18, R19, R2, R20, R22, R23, R24, R3, R4, R5, R6, R7, R8, R9: R, Resistors_SMD:R_0805, symbol R
- added R29: 10k, Resistors_SMD:R_0805, symbol R
- added U4: STM32F302C, symbol STM32F302C
- C3: renamed from C?; footprint (none) -> Capacitors_SMD:C_0805; Source (none) -> DigiKey
- D1, D2, D3, D4, D5, D7: renamed from D?; value LED_RABG -> RGB; Part (none) -> CLV1A-FKB-CK1N1G1BB7D4C3CT-ND; Source (none) -> DigiKey
- D8, D9: renamed from D?; value LED -> RED; footprint (none) -> Diodes_SMD:D_1206; Part (none) -> 160-1405-1-ND; Source (none) -> DigiKey
- R1, R30, R31: renamed from R?; footprint (none) -> Resistors_SMD:R_0805; Source (none) -> DigiKey
- gave numbers to parts that had none: 49
Connections:
- wire segments 235 -> 255
Other:
- moved on the sheet: C13, C14, C15, C16, C17, C18, C2, D8, F1, J2, J4, J5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

Commit message: Working on main board schematic
Parts:
- removed J10, J11, J12, J7, J8, J9: TP, Measurement_Points:Measurement_Point_Round-SMD-Pad_Big, symbol TEST_1P
- removed R13, R16, R29, R31: 10k, Resistors_SMD:R_0805, symbol R
- removed R32: R, symbol R
- added R19, R20, R21, R33, R35, R5, R8, R9: 10k, Resistors_SMD:R_0805, symbol R
- added R?: R, Resistors_SMD:R_0805, symbol R
- added SW1, SW2, SW3, SW4: SW_Push, Buttons_Switches_ThroughHole:SW_PUSH_6mm, symbol SW_Push
- added TP1, TP2, TP3, TP4, TP5, TP6: TP, Measurement_Points:Measurement_Point_Round-TH_Small, symbol TEST_1P
- BT1: footprint (none) -> radio-clock:S8411-45R; Part (none) -> 952-1745-1-ND; Source (none) -> DigiKey
- D6: value D -> MURS140; footprint (none) -> Diodes_SMD:D_SMB_Standard; Part (none) -> MURS140-FDICT-ND; Source (none) -> DigiKey
- J1: renamed from J2; footprint (none) -> radio-clock:PJ-002AH-SMT-TR; Part (none) -> CP-002AHPJCT-ND; Source (none) -> DigiKey
- J5: footprint (none) -> radio-clock:TC2050-IDC
- L1: footprint (none) -> radio-clock:B82477R4104M100; Part (none) -> 495-4547-1-ND; Source (none) -> DigiKey
- R13: renamed from R10; footprint (none) -> Resistors_SMD:R_0805; Part (none) -> 311-10.0KCRCT-ND; Source (none) -> DigiKey
- R15, R17: Part (none) -> 311-10.0KCRCT-ND
- U2: footprint (none) -> Housings_SOIC:SOIC-8_3.9x4.9mm_Pitch1.27mm; Part (none) -> MAX1771CSA+CT-ND; Source (none) -> DigiKey
- U3: footprint (none) -> radio-clock:FGPMMOPA6H; Part (none) -> 790; Source (none) -> Adafruit
- U4: footprint (none) -> Housings_QFP:LQFP-48_7x7mm_Pitch0.5mm; Part (none) -> 497-14699-ND; Source (none) -> DigiKey
- renumbered J1 to J2, R7 to R10, R8 to R11, R9 to R12, R11 to R14, R12 to R16, R14 to R18, R18 to R22, R19 to R23, R20 to R24, R21 to R25, R22 to R26, R23 to R27, R24 to R28, R25 to R29, R26 to R30, R27 to R31, R28 to R32, R30 to R34, R5 to R6, R6 to R7
Connections:
- net labels added: PB1, PB2, PB3, PB4
- net labels removed: NJTRST
- wire segments 255 -> 277
- no-connect marks 3 -> 5
Other:
- moved on the sheet: D1, D2, D3, D4, D5, D7, Q7, Q8, Q9, R1, R10, R11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

Commit message: Working on main board schematic
Parts:
- D1, D2, D3, D4, D5, D7: footprint (none) -> radio-clock:PLCC-4
- J2, J3: Part (none) -> A99476CT-ND
- J4: footprint (none) -> radio-clock:10118192; Part (none) -> 609-4613-1-ND; Source (none) -> DigiKey
- J6: footprint (none) -> Connect:SMA_THT_Jack_Straight; Part (none) -> CONSMA002-L-ND; Source (none) -> DigiKey
- JP1: footprint (none) -> Pin_Headers:Pin_Header_Straight_1x02_Pitch2.54mm; Part (none) -> 3M9447-ND; Source (none) -> DigiKey
- L2: footprint (none) -> Resistors_SMD:R_0805; Part (none) -> 490-1054-1-ND; Source (none) -> DigiKey
- gave numbers to parts that had none: 1
Changed lines of the file:
@@
 F 0 "J4" H 8050 1800 50  0000 L CNN
 F 1 "USB_OTG" H 8050 1700 50  0000 L CNN
-F 2 "" H 8400 1300 50  0001 C CNN
+F 2 "radio-clock:10118192" H 8400 1300 50  0001 C CNN
 F 3 "" H 8400 1300 50  0001 C CNN
+F 4 "DigiKey" H 8250 1350 60  0001 C CNN "Source"
+F 5 "609-4613-1-ND" H 8250 1350 60  0001 C CNN "Part"
 	1    8250 1350
 	1    0    0    -1
@@
 F 3 "" H 2000 2100 50  0001 C CNN
 F 4 "DigiKey" H 2000 2100 60  0001 C CNN "Source"
+F 5 "A99476CT-ND" H 2000 2100 60  0001 C CNN "Part"
 	1    2000 2100
 	-1   0    0    -1
@@
 F 3 "" H 6650 2100 50  0001 C CNN
 F 4 "DigiKey" H 6650 2100 60  0001 C CNN "Source"
+F 5 "A99476CT-ND" H 6650 2100 60  0001 C CNN "Part"
 	1    6650 2100
 	1    0    0    -1
@@
 F 0 "J6" H 14460 7470 50  0000 C CNN
 F 1 "SMA" H 14550 7200 50  0000 C CNN
-F 2 "" H 14450 7350 50  0001 C CNN
+F 2 "Connect:SMA_THT_Jack_Straight" H 14450 7350 50  0001 C CNN
 F 3 "" H 14450 7350 50  0001 C CNN
+F 4 "DigiKey" H 14450 7350 60  0001 C CNN "Source"
+F 5 "CONSMA002-L-ND" H 14450 7350 60  0001 C CNN "Part"
 	1    14450 7350
 	1    0    0    -1
@@
 F 0 "L2" V 11750 5500 50  0000 C CNN
 F 1 "FERRITE" V 11910 5500 50  0000 C CNN
-F 2 "" H 11800 5500 50  0001 C CNN
+F 2 "Resistors_SMD:R_0805" H 11800 5500 50  0001 C CNN
 F 3 "" H 11800 5500 50  0001 C CNN
+F 4 "DigiKey" H 11800 5500 60  0001 C CNN "Source"
+F 5 "490-1054-1-ND" H 11800 5500 60  0001 C CNN "Part"
 	1    11800 5500
 	0    -1   -1   0
@@
 F 0 "JP1" H 11250 2330 50  0000 C CNN
 F 1 "Jumper_NO_Small" H 11260 2190 50  0001 C CNN
-F 2 "" H 11250 2250 50  0001 C CNN
+F 2 "Pin_Headers:Pin_Header_Straight_1x02_Pitch2.54mm" H 11250 2250 50  0001 C CNN
 F 3 "" H 11250 2250 50  0001 C CNN
+F 4 "DigiKey" H 11250 2250 60  0001 C CNN "Source"
+F 5 "3M9447-ND" H 11250 2250 60  0001 C CNN "Part"
 	1    11250 2250
 	0    -1   -1   0
@@
 F 0 "D1" V 1650 4800 50  0000 C CNN
 F 1 "RGB" V 1650 4300 50  0000 C CNN
-F 2 "" H 1500 4500 50  0001 C CNN
+F 2 "radio-clock:PLCC-4" H 1500 4500 50  0001 C CNN
 F 3 "" H 1500 4500 50  0001 C CNN
 F 4 "DigiKey" H 1500 4550 60  0001 C CNN "Source"
@@
 	1    1500 4300
 	1    0    0    -1
-$EndComp
-$Comp
-L LED_RABG D2
-U 1 1 58E654AC
-P 2350 4550
-F 0 "D2" V 2500 4800 50  0000 C CNN
-F 1 "RGB" V 2500 4300 50  0000 C CNN
-F 2 "" H 2350 4500 50  0001 C CNN
-F 3 "" H 2350 4500 50  0001 C CNN
-F 4 "DigiKey" H 2350 4550 60  0001 C CNN "Source"
-F 5 "CLV1A-FKB-CK1N1G1BB7D4C3CT-ND" H 2350 4550 60  0001 C CNN "Part"
-	1    2350 4550
-	0    -1   -1   0
-$EndComp
-$Comp
-L LED_RABG D3
-U 1 1 58E65572
-P 3800 4550
-F 0 "D3" V 3950 4800 50  0000 C CNN
-F 1 "RGB" V 3950 4300 50  0000 C CNN
-F 2 "" H 3800 4500 50  0001 C CNN
-F 3 "" H 3800 4500 50  0001 C CNN
-F 4 "DigiKey" H 3800 4550 60  0001 C CNN "Source"
-F 5 "CLV1A-FKB-CK1N1G1BB7D4C3CT-ND" H 3800 4550 60  0001 C CNN "Part"
-	1    3800 4550
-	0    -1   -1   0
-$EndComp
-$Comp
-L LED_RABG D4
-U 1 1 58E65639
-P 4650 4550
-F 0 "D4" V 4800 4800 50  0000 C CNN
-F 1 "RGB" V 4800 4300 50  0000 C CNN
-F 2 "" H 4650 4500 50  0001 C CNN
-F 3 "" H 4650 4500 50  0001 C CNN
-F 4 "DigiKey" H 4650 4550 60  0001 C CNN "Source"
-F 5 "CLV1A-FKB-CK1N1G1BB7D4C3CT-ND" H 4650 4550 60  0001 C CNN "Part"
-	1    4650 4550
-	0    -1   -1   0
-$EndComp
-$Comp
-L LED_RABG D5
-U 1 1 58E6582B
-P 6100 4550
-F 0 "D5" V 6250 4800 50  0000 C CNN
-F 1 "RGB" V 6250 4300 50  0000 C CNN
-F 2 "" H 6100 4500 50  0001 C CNN
-F 3 "" H 6100 4500 50  0001 C CNN
-F 4 "DigiKey" H 6100 4550 60  0001 C CNN "Source"
-F 5 "CLV1A-FKB-CK1N1G1BB7D4C3CT-ND" H 6100 4550 60  0001 C CNN "Part"
-	1    6100 4550
-	0    -1   -1   0
-$EndComp
-$Comp
-L LED_RABG D7
-U 1 1 58E65AAF
-P 6950 4550
-F 0 "D7" V 7100 4800 50  0000 C CNN
-F 1 "RGB" V 7100 4300 50  0000 C CNN
-F 2 "" H 6950 4500 50  0001 C CNN
-F 3 "" H 6950 4500 50  0001 C CNN
-F 4 "DigiKey" H 6950 4550 60  0001 C CNN "Source"
-F 5 "CLV1A-FKB-CK1N1G1BB7D4C3CT-ND" H 6950 4550 60  0001 C CNN "Part"
-	1    6950 4550
-	0    -1   -1   0
 $EndComp
 $Comp
@@
 $EndComp
 $Comp
-L R R?
+L R R36
 U 1 1 58E8F0D9
 P 13800 6350
-F 0 "R?" V 13880 6350 50  0000 C CNN
+F 0 "R36" V 13880 6350 50  0000 C CNN
 F 1 "R" V 13800 6350 50  0000 C CNN
 F 2 "Resistors_SMD:R_0805" V 13730 6350 50  0001 C CNN
@@
 NoConn ~ 8050 3150
 NoConn ~ 14750 2450
+$Comp
+L LED_RABG D2
+U 1 1 58E85C8B
+P 2350 4550
+F 0 "D2" V 2500 4800 50  0000 C CNN
+F 1 "RGB" V 2500 4300 50  0000 C CNN
+F 2 "radio-clock:PLCC-4" H 2350 4500 50  0001 C CNN
+F 3 "" H 2350 4500 50  0001 C CNN
+F 4 "DigiKey" H 2350 4550 60  0001 C CNN "Source"
+F 5 "CLV1A-FKB-CK1N1G1BB7D4C3CT-ND" H 2350 4550 60  0001 C CNN "Part"
+	1    2350 4550
+	0    -1   -1   0
+$EndComp
+$Comp
+L LED_RABG D3
+U 1 1 58E85DC9
+P 3800 4550
+F 0 "D3" V 3950 4800 50  0000 C CNN
+F 1 "RGB" V 3950 4300 50  0000 C CNN
+F 2 "radio-clock:PLCC-4" H 3800 4500 50  0001 C CNN
+F 3 "" H 3800 4500 50  0001 C CNN
+F 4 "DigiKey" H 3800 4550 60  0001 C CNN "Source"
+F 5 "CLV1A-FKB-CK1N1G1BB7D4C3CT-ND" H 3800 4550 60  0001 C CNN "Part"
+	1    3800 4550
+	0    -1   -1   0
+$EndComp
+$Comp
+L LED_RABG D4
+U 1 1 58E85F10
+P 4650 4550
+F 0 "D4" V 4800 4800 50  0000 C CNN
+F 1 "RGB" V 4800 4300 50  0000 C CNN
+F 2 "radio-clock:PLCC-4" H 4650 4500 50  0001 C CNN
+F 3 "" H 4650 4500 50  0001 C CNN
+F 4 "DigiKey" H 4650 4550 60  0001 C CNN "Source"
+F 5 "CLV1A-FKB-CK1N1G1BB7D4C3CT-ND" H 4650 4550 60  0001 C CNN "Part"
+	1    4650 4550
+	0    -1   -1   0
+$EndComp
+$Comp
+L LED_RABG D5
+U 1 1 58E8604C
+P 6100 4550
+F 0 "D5" V 6250 4800 50  0000 C CNN
+F 1 "RGB" V 6250 4300 50  0000 C CNN
+F 2 "radio-clock:PLCC-4" H 6100 4500 50  0001 C CNN
+F 3 "" H 6100 4500 50  0001 C CNN
+F 4 "DigiKey" H 6100 4550 60  0001 C CNN "Source"
+F 5 "CLV1A-FKB-CK1N1G1BB7D4C3CT-ND" H 6100 4550 60  0001 C CNN "Part"
+	1    6100 4550
+	0    -1   -1   0
+$EndComp
+$Comp
+L LED_RABG D7
+U 1 1 58E8618F
+P 6950 4550
+F 0 "D7" V 7100 4800 50  0000 C CNN
+F 1 "RGB" V 7100 4300 50  0000 C CNN
+F 2 "radio-clock:PLCC-4" H 6950 4500 50  0001 C CNN
+F 3 "" H 6950 4500 50  0001 C CNN
+F 4 "DigiKey" H 6950 4550 60  0001 C CNN "Source"
+F 5 "CLV1A-FKB-CK1N1G1BB7D4C3CT-ND" H 6950 4550 60  0001 C CNN "Part"
+	1    6950 4550
+	0    -1   -1   0
+$EndComp
 $EndSCHEMATC

Commit message: Working on main board schematic
Parts:
- removed C12: 0.1u, Capacitors_SMD:C_0603, symbol C
- added C11: 0.1u, Capacitors_SMD:C_0603, symbol C
- added C19, C20: C, symbol C
- added Y2: 32.768kHz, symbol Crystal
- C1, C3, C7: footprint Capacitors_SMD:C_0805 -> Capacitors_SMD:C_0603; Part (none) -> 311-1344-1-ND
- C14, C15: Part (none) -> 311-1344-1-ND
- C9: renamed from C11; Part (none) -> 311-1344-1-ND
- renumbered C9 to C10, C10 to C12, U4 to U3, U3 to U4
Connections:
- wire segments 277 -> 285
Other:
- moved on the sheet: BT1, C10, C12, C13, C16, C17, C18, C8, C9, D8, D9, J4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

Commit message: Working on main board schematic
Parts:
- removed D1, D2, D3, D4, D5, D7: RGB, radio-clock:PLCC-4, symbol LED_RABG
- removed R1, R10, R11, R12, R14, R18, R2, R26, R27, R28, R3, R4: R, Resistors_SMD:R_0805, symbol R
- added D1, D2, D3, D4, D5, D6: LED_BGR, radio-clock:PLCC-6, symbol LED_BGR
- added R15, R5: 1.05k, Resistors_SMD:R_0805, symbol R
- added R17: 499, Resistors_SMD:R_0805, symbol R
- R1: renamed from R22; value R -> 1.05k
- R16, R6: value R -> 2.43k
- R2: renamed from R23; value R -> 2.43k
- R3: renamed from R24; value R -> 499
- R7: value R -> 499
- renumbered D6 to D7, R13 to R10, R17 to R11, R15 to R12, R19 to R13, R20 to R14, R21 to R18, R25 to R19, R29 to R20, R30 to R21, R31 to R22, R32 to R23, R33 to R24, R34 to R25, R35 to R26, R36 to R27, R5 to R4
Connections:
- wire segments 285 -> 360
Other:
- moved on the sheet: R1, R12, R2, R3, R4, R8, R9, SW1, SW2, SW3, SW4
