File: hardware/tube-board/tube-board.sch (KiCad schematic (older format))
At the start: 18 parts, among them J1 CONN_01X10, J2 CONN_01X10, U1 HV5522PG, U2 HV5522PG

Commit message: Completed BOMs for both boards
Parts:
- AN1, AN2, AN3, AN4, AN5, AN6: Source DigiKey -> eBay
- C1, C2: Part (none) -> 311-1136-1-ND
- U1, U2: Part (none) -> 689-HV5522PG-G; Source DigiKey -> Mouser
Changed lines of the file:
@@
 EESchema Schematic File Version 2
-LIBS:tube-board-rescue
 LIBS:power
 LIBS:device
@@
 F 2 "Housings_QFP:LQFP-44_10x10mm_Pitch0.8mm" H 9850 5450 60  0001 C CNN
 F 3 "" H 9850 5450 60  0001 C CNN
-F 4 "DigiKey" H 9850 5450 60  0001 C CNN "Source"
+F 4 "Mouser" H 9850 5450 60  0001 C CNN "Source"
+F 5 "689-HV5522PG-G" H 9850 5450 60  0001 C CNN "Part"
 	1    9850 5450
 	1    0    0    -1
@@
 F 2 "Housings_QFP:LQFP-44_10x10mm_Pitch0.8mm" H 4650 5450 60  0001 C CNN
 F 3 "" H 4650 5450 60  0001 C CNN
-F 4 "DigiKey" H 4650 5450 60  0001 C CNN "Source"
+F 4 "Mouser" H 4650 5450 60  0001 C CNN "Source"
+F 5 "689-HV5522PG-G" H 4650 5450 60  0001 C CNN "Part"
 	1    4650 5450
 	1    0    0    -1
@@
 F 2 "radio-clock:IN-14" H 2300 1950 60  0001 C CNN
 F 3 "" H 2300 1950 60  0001 C CNN
-F 4 "DigiKey" H 2300 1950 60  0001 C CNN "Source"
+F 4 "eBay" H 2300 1950 60  0001 C CNN "Source"
 	1    2300 1950
 	1    0    0    -1
@@
 F 2 "radio-clock:IN-14" H 4200 1950 60  0001 C CNN
 F 3 "" H 4200 1950 60  0001 C CNN
-F 4 "DigiKey" H 4200 1950 60  0001 C CNN "Source"
+F 4 "eBay" H 4200 1950 60  0001 C CNN "Source"
 	1    4200 1950
 	1    0    0    -1
@@
 F 2 "radio-clock:IN-14" H 7500 1950 60  0001 C CNN
 F 3 "" H 7500 1950 60  0001 C CNN
-F 4 "DigiKey" H 7500 1950 60  0001 C CNN "Source"
+F 4 "eBay" H 7500 1950 60  0001 C CNN "Source"
 	1    7500 1950
 	1    0    0    -1
@@
 F 2 "radio-clock:IN-14" H 9400 1950 60  0001 C CNN
 F 3 "" H 9400 1950 60  0001 C CNN
-F 4 "DigiKey" H 9400 1950 60  0001 C CNN "Source"
+F 4 "eBay" H 9400 1950 60  0001 C CNN "Source"
 	1    9400 1950
 	1    0    0    -1
@@
 F 2 "radio-clock:IN-14" H 12700 1950 60  0001 C CNN
 F 3 "" H 12700 1950 60  0001 C CNN
-F 4 "DigiKey" H 12700 1950 60  0001 C CNN "Source"
+F 4 "eBay" H 12700 1950 60  0001 C CNN "Source"
 	1    12700 1950
 	1    0    0    -1
@@
 F 2 "radio-clock:IN-14" H 14600 1950 60  0001 C CNN
 F 3 "" H 14600 1950 60  0001 C CNN
-F 4 "DigiKey" H 14600 1950 60  0001 C CNN "Source"
+F 4 "eBay" H 14600 1950 60  0001 C CNN "Source"
 	1    14600 1950
 	1    0    0    -1
@@
 F 3 "" H 2900 4000 50  0001 C CNN
 F 4 "DigiKey" H 2900 4000 60  0001 C CNN "Source"
+F 5 "311-1136-1-ND" H 2900 4000 60  0001 C CNN "Part"
 	1    2900 4000
 	1    0    0    -1
@@
 F 3 "" H 8000 4050 50  0001 C CNN
 F 4 "DigiKey" H 8000 4050 60  0001 C CNN "Source"
+F 5 "311-1136-1-ND" H 8000 4050 60  0001 C CNN "Part"
 	1    8000 4050
 	1    0    0    -1

Commit message: Fixed BOM part number error on tube-board
Parts:
- C1, C2: Part 311-1136-1-ND -> 311-1140-1-ND
Changed lines of the file:
@@
 F 3 "" H 2900 4000 50  0001 C CNN
 F 4 "DigiKey" H 2900 4000 60  0001 C CNN "Source"
-F 5 "311-1136-1-ND" H 2900 4000 60  0001 C CNN "Part"
+F 5 "311-1140-1-ND" H 2900 4000 60  0001 C CNN "Part"
 	1    2900 4000
 	1    0    0    -1
@@
 F 3 "" H 8000 4050 50  0001 C CNN
 F 4 "DigiKey" H 8000 4050 60  0001 C CNN "Source"
-F 5 "311-1136-1-ND" H 8000 4050 60  0001 C CNN "Part"
+F 5 "311-1140-1-ND" H 8000 4050 60  0001 C CNN "Part"
 	1    8000 4050
 	1    0    0    -1
